File: Hardware/Schematics/04-Pilotaggio Matrice/04-Pilotaggio Matrice.kicad_sch (KiCad schematic)
At the start: 10 parts, among them U1 CD74HC4067M, U2 CD74HC4067M, U3 CD74HC4067M, U69A AD8604ARUZ

Commit message: update
Parts:
- added C183, C49, C51, C53: 100nF, symbol Device:C
- added J2: Conn_02x32_Odd_Even, Connector_PinHeader_1.00mm:PinHeader_2x32_P1.00mm_Vertical, symbol Connector_Generic:Conn_02x32_Odd_Even
- added TP-EN1, TP-EN2, TP-EN3, TP-R0, TP-R1, TP-R2, TP-R3: TestPoint, symbol Connector:TestPoint
- added U4: CD74HC4067M, Package_SO:SOIC-24W_7.5x15.4mm_P1.27mm, symbol 74xx:CD74HC4067M
Connections:
- net +5V: now also U1.24 (VCC), U2.24 (VCC), U3.24 (VCC), C183.2, C49.2, C51.2, C53.2, U4.24 (VCC)
- net GNDREF: now reaches U1.1 (COM)
- net GNDREF: now also U1.12 (GND), U2.1 (COM), U2.12 (GND), U3.1 (COM), U3.12 (GND), C183.1, C49.1, C51.1, C53.1, U4.1 (COM), U4.12 (GND)
- net COL0: now reaches U1.10 (S0)
- net COL0: now also U2.10 (S0), U3.10 (S0), TP-R0.1, U4.10 (S0)
- net COL1: now reaches U1.11 (S1)
- net COL1: now also U2.11 (S1), U3.11 (S1), TP-R1.1, U4.11 (S1)
- net COL3: now reaches U1.13 (S3)
- net COL3: now also U2.13 (S3), U3.13 (S3), TP-R3.1, U4.13 (S3)
- net COL2: now reaches U1.14 (S2)
- net COL2: now also U2.14 (S2), U3.14 (S2), TP-R2.1, U4.14 (S2)
- net EN-COL-01-16: now reaches U1.15 (~{E})
- net EN-COL-01-16: now also TP-EN1.1
- net X16: now reaches U1.16 (I15)
- net X16: now also J2.16 (Pin_16)
- net X15: now reaches U1.17 (I14)
- net X15: now also J2.15 (Pin_15)
- net X14: now reaches U1.18 (I13)
- net X13: now reaches U1.19 (I12)
- net X13: now also J2.13 (Pin_13)
- net X8: now reaches U1.2 (I7)
- net X12: now reaches U1.20 (I11)
- net X11: now reaches U1.21 (I10)
- net X11: now also J2.11 (Pin_11)
- net X10: now reaches U1.22 (I9)
- net X9: now reaches U1.23 (I8)
- net X9: now also J2.9 (Pin_9)
- net X7: now reaches U1.3 (I6)
- net X7: now also J2.7 (Pin_7)
- net X6: now reaches U1.4 (I5)
- net X5: now reaches U1.5 (I4)
- net X5: now also J2.5 (Pin_5)
- net X4: now reaches U1.6 (I3)
- net X3: now reaches U1.7 (I2)
- net X3: now also J2.3 (Pin_3)
- net X2: now reaches U1.8 (I1)
- net X2: now also J2.2 (Pin_2)
- net X1: now reaches U1.9 (I0)
- net X1: now also J2.1 (Pin_1)
- net EN-COL-17-32: now reaches U2.15 (~{E})
- net EN-COL-17-32: now also TP-EN2.1
- net X32: now reaches U2.16 (I15)
- net X31: now reaches U2.17 (I14)
- net X30: now reaches U2.18 (I13)
- net X29: now reaches U2.19 (I12)
- net X24: now reaches U2.2 (I7)
- net X28: now reaches U2.20 (I11)
- net X27: now reaches U2.21 (I10)
- net X26: now reaches U2.22 (I9)
- net X25: now reaches U2.23 (I8)
- net X23: now reaches U2.3 (I6)
- net X22: now reaches U2.4 (I5)
- net X21: now reaches U2.5 (I4)
- net X20: now reaches U2.6 (I3)
- net X19: now reaches U2.7 (I2)
- net X18: now reaches U2.8 (I1)
- net X17: now reaches U2.9 (I0)
- net X17: now also J2.17 (Pin_17)
- net EN-COL-33-48: now reaches U3.15 (~{E})
- net EN-COL-33-48: now also TP-EN3.1
- net X48: now reaches U3.16 (I15)
- net X47: now reaches U3.17 (I14)
- net X46: now reaches U3.18 (I13)
- net X45: now reaches U3.19 (I12)
- net X40: now reaches U3.2 (I7)
- net X44: now reaches U3.20 (I11)
- net X43: now reaches U3.21 (I10)
- net X42: now reaches U3.22 (I9)
- net X41: now reaches U3.23 (I8)
- net X39: now reaches U3.3 (I6)
- net X38: now reaches U3.4 (I5)
- net X37: now reaches U3.5 (I4)
- net X36: now reaches U3.6 (I3)
- net X35: now reaches U3.7 (I2)
- net X34: now reaches U3.8 (I1)
- net X33: now reaches U3.9 (I0)
- new net EN-COL-49-64: U4.15 (~{E})
- new net X49: U4.9 (I0)
- new net X50: U4.8 (I1)
- new net X51: U4.7 (I2)
- new net X52: U4.6 (I3)
- new net X53: U4.5 (I4)
- new net X54: U4.4 (I5)
- new net X55: U4.3 (I6)
- new net X56: U4.2 (I7)
- new net X57: U4.23 (I8)
- new net X58: U4.22 (I9)
- new net X59: U4.21 (I10)
- new net X60: U4.20 (I11)
- new net X61: U4.19 (I12)
- new net X62: U4.18 (I13)
- new net X63: U4.17 (I14)
- new net X64: U4.16 (I15)
Other:
- moved on the sheet: U1

Commit message: update
Parts:
- added C1, C10, C100, C101, C11, C12, C14, C16, C17, C18, C19, C2, C20, C21, C22, C24, C26, C27, C28, C29, C3, C30, C31, C32, C34, C36, C37, C38, C39, C4, C40, C41, C42, C44, C46, C47, C48, C5, C50, C52, C54, C55, C57, C59, C6, C60, C61, C62, C63, C64, C65, C67, C69, C7, C70, C71, C72, C73, C74, C75, C77, C79, C8, C80, C81, C82, C83, C84, C85, C87, C89, C9, C90, C91, C92, C93, C94, C95, C97, C99: 56pF, symbol Device:C
- added C13, C15, C2, C23, C25, C33, C35, C43, C45, C56, C58, C66, C68, C7, C76, C78, C86, C88, C96, C98: 100nF, symbol Device:C
- added R1, R10, R11, R12, R13, R14, R15, R16, R17, R18, R19, R2, R20, R21, R22, R23, R24, R25, R26, R27, R28, R29, R3, R30, R31, R32, R33, R34, R35, R36, R37, R38, R39, R4, R40, R41, R42, R43, R44, R45, R46, R47, R48, R49, R5, R50, R51, R52, R53, R54, R55, R56, R57, R58, R59, R6, R60, R61, R62, R63, R64, R65, R66, R67, R68, R69, R7, R70, R71, R72, R73, R74, R75, R76, R77, R78, R79, R8, R80, R9: 560, symbol Device:R_US
- added U10, U11, U12, U13, U14, U15, U16, U17, U18, U19, U20, U21, U22, U23, U24, U25, U26, U5, U6, U7, U8, U9: AD8604ARUZ, AD8604ARUZ:SOP65P640X120-14N, symbol AD8604ARUZ:AD8604ARUZ
Connections:
- net +5V: now also C13.2, C15.2, C2.2, C23.2, C25.2, C33.2, C35.2, C43.2, C45.2, C56.2, C58.2, C66.2, C68.2, C7.2, C76.2, C78.2, C86.2, C88.2, C96.2, C98.2, U10.4 (V+), U11.4 (V+), U12.4 (V+), U13.4 (V+), U14.4 (V+), U15.4 (V+), U16.4 (V+), U17.4 (V+), U18.4 (V+), U19.4 (V+), U20.4 (V+), U21.4 (V+), U22.4 (V+), U23.4 (V+), U24.4 (V+), U25.4 (V+), U26.4 (V+), U7.4 (V+), U8.4 (V+), U9.4 (V+)
- net GND: now also C13.1, C15.1, C2.1, C23.1, C25.1, C33.1, C35.1, C43.1, C45.1, C56.1, C58.1, C66.1, C68.1, C7.1, C76.1, C78.1, C86.1, C88.1, C96.1, C98.1, U10.11 (V-), U11.11 (V-), U12.11 (V-), U13.11 (V-), U14.11 (V-), U15.11 (V-), U16.11 (V-), U17.11 (V-), U18.11 (V-), U19.11 (V-), U20.11 (V-), U21.11 (V-), U22.11 (V-), U23.11 (V-), U24.11 (V-), U25.11 (V-), U26.11 (V-), U7.11 (V-), U8.11 (V-), U9.11 (V-)
- net Vr: now also U10.10 (+IN_C), U10.12 (+IN_D), U10.3 (+IN_A), U10.5 (+IN_B), U11.10 (+IN_C), U11.12 (+IN_D), U11.3 (+IN_A), U11.5 (+IN_B), U12.10 (+IN_C), U12.12 (+IN_D), U12.3 (+IN_A), U12.5 (+IN_B), U13.10 (+IN_C), U13.12 (+IN_D), U13.3 (+IN_A), U13.5 (+IN_B), U14.10 (+IN_C), U14.12 (+IN_D), U14.3 (+IN_A), U14.5 (+IN_B), U15.10 (+IN_C), U15.12 (+IN_D), U15.3 (+IN_A), U15.5 (+IN_B), U16.10 (+IN_C), U16.12 (+IN_D), U16.3 (+IN_A), U16.5 (+IN_B), U17.10 (+IN_C), U17.12 (+IN_D), U17.3 (+IN_A), U17.5 (+IN_B), U18.10 (+IN_C), U18.12 (+IN_D), U18.3 (+IN_A), U18.5 (+IN_B), U19.10 (+IN_C), U19.12 (+IN_D), U19.3 (+IN_A), U19.5 (+IN_B), U20.10 (+IN_C), U20.12 (+IN_D), U20.3 (+IN_A), U20.5 (+IN_B), U21.10 (+IN_C), U21.12 (+IN_D), U21.3 (+IN_A), U21.5 (+IN_B), U22.10 (+IN_C), U22.12 (+IN_D), U22.3 (+IN_A), U22.5 (+IN_B), U23.10 (+IN_C), U23.12 (+IN_D), U23.3 (+IN_A), U23.5 (+IN_B), U24.10 (+IN_C), U24.12 (+IN_D), U24.3 (+IN_A), U24.5 (+IN_B), U25.10 (+IN_C), U25.12 (+IN_D), U25.3 (+IN_A), U25.5 (+IN_B), U26.10 (+IN_C), U26.12 (+IN_D), U26.3 (+IN_A), U26.5 (+IN_B), U7.10 (+IN_C), U7.12 (+IN_D), U7.3 (+IN_A), U7.5 (+IN_B), U8.10 (+IN_C), U8.12 (+IN_D), U8.3 (+IN_A), U8.5 (+IN_B), U9.10 (+IN_C), U9.12 (+IN_D), U9.3 (+IN_A), U9.5 (+IN_B)
- new net AY1: C1.2, C14.2, C24.2, C34.2, C44.2, C57.2, C67.2, C77.2, C87.2, C97.2, R1.2, R13.2, R21.2, R29.2, R37.2, R45.2, R53.2, R61.2, R69.2, R77.2, U11.1 (OUT_A), U13.1 (OUT_A), U15.1 (OUT_A), U17.1 (OUT_A), U19.1 (OUT_A), U21.1 (OUT_A), U23.1 (OUT_A), U25.1 (OUT_A), U7.1 (OUT_A), U9.1 (OUT_A)
- new net AY2: C19.2, C2.2, C29.2, C39.2, C50.2, C62.2, C72.2, C82.2, C9.2, C92.2, R17.2, R2.2, R25.2, R33.2, R41.2, R49.2, R57.2, R65.2, R73.2, R9.2, U11.7 (OUT_B), U13.7 (OUT_B), U15.7 (OUT_B), U17.7 (OUT_B), U19.7 (OUT_B), U21.7 (OUT_B), U23.7 (OUT_B), U25.7 (OUT_B), U7.7 (OUT_B), U9.7 (OUT_B)
- new net AY3: C100.2, C17.2, C27.2, C3.2, C37.2, C47.2, C60.2, C70.2, C80.2, C90.2, R15.2, R23.2, R3.2, R31.2, R39.2, R47.2, R55.2, R63.2, R71.2, R79.2, U11.8 (OUT_C), U13.8 (OUT_C), U15.8 (OUT_C), U17.8 (OUT_C), U19.8 (OUT_C), U21.8 (OUT_C), U23.8 (OUT_C), U25.8 (OUT_C), U7.8 (OUT_C), U9.8 (OUT_C)
- new net AY4: C10.2, C20.2, C30.2, C4.2, C40.2, C52.2, C63.2, C73.2, C83.2, C93.2, R10.2, R18.2, R26.2, R34.2, R4.2, R42.2, R50.2, R58.2, R66.2, R74.2, U11.14 (OUT_D), U13.14 (OUT_D), U15.14 (OUT_D), U17.14 (OUT_D), U19.14 (OUT_D), U21.14 (OUT_D), U23.14 (OUT_D), U25.14 (OUT_D), U7.14 (OUT_D), U9.14 (OUT_D)
- new net AY5: C16.2, C26.2, C36.2, C46.2, C5.2, C59.2, C69.2, C79.2, C89.2, C99.2, R14.2, R22.2, R30.2, R38.2, R46.2, R5.2, R54.2, R62.2, R70.2, R78.2, U10.1 (OUT_A), U12.1 (OUT_A), U14.1 (OUT_A), U16.1 (OUT_A), U18.1 (OUT_A), U20.1 (OUT_A), U22.1 (OUT_A), U24.1 (OUT_A), U26.1 (OUT_A), U8.1 (OUT_A)
- new net AY6: C11.2, C21.2, C31.2, C41.2, C54.2, C6.2, C64.2, C74.2, C84.2, C94.2, R11.2, R19.2, R27.2, R35.2, R43.2, R51.2, R59.2, R6.2, R67.2, R75.2, U10.7 (OUT_B), U12.7 (OUT_B), U14.7 (OUT_B), U16.7 (OUT_B), U18.7 (OUT_B), U20.7 (OUT_B), U22.7 (OUT_B), U24.7 (OUT_B), U26.7 (OUT_B), U8.7 (OUT_B)
- new net AY7: C101.2, C18.2, C28.2, C38.2, C48.2, C61.2, C7.2, C71.2, C81.2, C91.2, R16.2, R24.2, R32.2, R40.2, R48.2, R56.2, R64.2, R7.2, R72.2, R80.2, U10.8 (OUT_C), U12.8 (OUT_C), U14.8 (OUT_C), U16.8 (OUT_C), U18.8 (OUT_C), U20.8 (OUT_C), U22.8 (OUT_C), U24.8 (OUT_C), U26.8 (OUT_C), U8.8 (OUT_C)
- new net AY8: C12.2, C22.2, C32.2, C42.2, C55.2, C65.2, C75.2, C8.2, C85.2, C95.2, R12.2, R20.2, R28.2, R36.2, R44.2, R52.2, R60.2, R68.2, R76.2, R8.2, U10.14 (OUT_D), U12.14 (OUT_D), U14.14 (OUT_D), U16.14 (OUT_D), U18.14 (OUT_D), U20.14 (OUT_D), U22.14 (OUT_D), U24.14 (OUT_D), U26.14 (OUT_D), U8.14 (OUT_D)
- new net Y1: C1.1, C14.1, C24.1, C34.1, C44.1, C57.1, C67.1, C77.1, C87.1, C97.1, R1.1, R13.1, R21.1, R29.1, R37.1, R45.1, R53.1, R61.1, R69.1, R77.1, U11.2 (-IN_A), U13.2 (-IN_A), U15.2 (-IN_A), U17.2 (-IN_A), U19.2 (-IN_A), U21.2 (-IN_A), U23.2 (-IN_A), U25.2 (-IN_A), U7.2 (-IN_A), U9.2 (-IN_A)
- new net Y2: C19.1, C2.1, C29.1, C39.1, C50.1, C62.1, C72.1, C82.1, C9.1, C92.1, R17.1, R2.1, R25.1, R33.1, R41.1, R49.1, R57.1, R65.1, R73.1, R9.1, U11.6 (-IN_B), U13.6 (-IN_B), U15.6 (-IN_B), U17.6 (-IN_B), U19.6 (-IN_B), U21.6 (-IN_B), U23.6 (-IN_B), U25.6 (-IN_B), U7.6 (-IN_B), U9.6 (-IN_B)
- new net Y3: C100.1, C17.1, C27.1, C3.1, C37.1, C47.1, C60.1, C70.1, C80.1, C90.1, R15.1, R23.1, R3.1, R31.1, R39.1, R47.1, R55.1, R63.1, R71.1, R79.1, U11.9 (-IN_C), U13.9 (-IN_C), U15.9 (-IN_C), U17.9 (-IN_C), U19.9 (-IN_C), U21.9 (-IN_C), U23.9 (-IN_C), U25.9 (-IN_C), U7.9 (-IN_C), U9.9 (-IN_C)
- new net Y4: C10.1, C20.1, C30.1, C4.1, C40.1, C52.1, C63.1, C73.1, C83.1, C93.1, R10.1, R18.1, R26.1, R34.1, R4.1, R42.1, R50.1, R58.1, R66.1, R74.1, U11.13 (-IN_D), U13.13 (-IN_D), U15.13 (-IN_D), U17.13 (-IN_D), U19.13 (-IN_D), U21.13 (-IN_D), U23.13 (-IN_D), U25.13 (-IN_D), U7.13 (-IN_D), U9.13 (-IN_D)
- new net Y5: C16.1, C26.1, C36.1, C46.1, C5.1, C59.1, C69.1, C79.1, C89.1, C99.1, R14.1, R22.1, R30.1, R38.1, R46.1, R5.1, R54.1, R62.1, R70.1, R78.1, U10.2 (-IN_A), U12.2 (-IN_A), U14.2 (-IN_A), U16.2 (-IN_A), U18.2 (-IN_A), U20.2 (-IN_A), U22.2 (-IN_A), U24.2 (-IN_A), U26.2 (-IN_A), U8.2 (-IN_A)
- new net Y6: C11.1, C21.1, C31.1, C41.1, C54.1, C6.1, C64.1, C74.1, C84.1, C94.1, R11.1, R19.1, R27.1, R35.1, R43.1, R51.1, R59.1, R6.1, R67.1, R75.1, U10.6 (-IN_B), U12.6 (-IN_B), U14.6 (-IN_B), U16.6 (-IN_B), U18.6 (-IN_B), U20.6 (-IN_B), U22.6 (-IN_B), U24.6 (-IN_B), U26.6 (-IN_B), U8.6 (-IN_B)
- new net Y7: C101.1, C18.1, C28.1, C38.1, C48.1, C61.1, C7.1, C71.1, C81.1, C91.1, R16.1, R24.1, R32.1, R40.1, R48.1, R56.1, R64.1, R7.1, R72.1, R80.1, U10.9 (-IN_C), U12.9 (-IN_C), U14.9 (-IN_C), U16.9 (-IN_C), U18.9 (-IN_C), U20.9 (-IN_C), U22.9 (-IN_C), U24.9 (-IN_C), U26.9 (-IN_C), U8.9 (-IN_C)
- new net Y8: C12.1, C22.1, C32.1, C42.1, C55.1, C65.1, C75.1, C8.1, C85.1, C95.1, R12.1, R20.1, R28.1, R36.1, R44.1, R52.1, R60.1, R68.1, R76.1, R8.1, U10.13 (-IN_D), U12.13 (-IN_D), U14.13 (-IN_D), U16.13 (-IN_D), U18.13 (-IN_D), U20.13 (-IN_D), U22.13 (-IN_D), U24.13 (-IN_D), U26.13 (-IN_D), U8.13 (-IN_D)

Commit message: update
Parts:
- removed C101, C71, C74, C75, C79, C81, C84, C85, C89, C91, C94, C95, C99: 56pF, symbol Device:C
- removed C78, C88, C98: 100nF, symbol Device:C
- removed R51, R52, R54, R56, R59, R60, R62, R64, R67, R68, R70, R72, R75, R76, R78, R80: 560, symbol Device:R_US
- removed U20, U22, U24, U26, U5, U6: AD8604ARUZ, AD8604ARUZ:SOP65P640X120-14N, symbol AD8604ARUZ:AD8604ARUZ
- added U20, U22, U5, U6: CD74HC4067M, Package_SO:SOIC-24W_7.5x15.4mm_P1.27mm, symbol 74xx:CD74HC4067M
- C64, C65, C69: value 56pF -> 100nF
Connections:
- net +5V: now also C64.2, C65.2, C69.2, U20.24 (VCC), U22.24 (VCC), U5.24 (VCC), U6.24 (VCC)
- net AY1: now also U6.9 (I0); no longer C14.2, C24.2, C34.2, C44.2, C57.2, C67.2, C77.2, C87.2, C97.2, R13.2, R21.2, R29.2, R37.2, R45.2, R53.2, R61.2, R69.2, R77.2, U11.1 (OUT_A), U13.1 (OUT_A), U15.1 (OUT_A), U17.1 (OUT_A), U19.1 (OUT_A), U21.1 (OUT_A), U23.1 (OUT_A), U25.1 (OUT_A), U9.1 (OUT_A)
- net AY2: now also U6.8 (I1); no longer C19.2, C29.2, C39.2, C50.2, C62.2, C72.2, C82.2, C9.2, C92.2, R17.2, R25.2, R33.2, R41.2, R49.2, R57.2, R65.2, R73.2, R9.2, U11.7 (OUT_B), U13.7 (OUT_B), U15.7 (OUT_B), U17.7 (OUT_B), U19.7 (OUT_B), U21.7 (OUT_B), U23.7 (OUT_B), U25.7 (OUT_B), U9.7 (OUT_B)
- net AY3: now also U6.7 (I2); no longer C100.2, C17.2, C27.2, C37.2, C47.2, C60.2, C70.2, C80.2, C90.2, R15.2, R23.2, R31.2, R39.2, R47.2, R55.2, R63.2, R71.2, R79.2, U11.8 (OUT_C), U13.8 (OUT_C), U15.8 (OUT_C), U17.8 (OUT_C), U19.8 (OUT_C), U21.8 (OUT_C), U23.8 (OUT_C), U25.8 (OUT_C), U9.8 (OUT_C)
- net AY4: now also U6.6 (I3); no longer C10.2, C20.2, C30.2, C40.2, C52.2, C63.2, C73.2, C83.2, C93.2, R10.2, R18.2, R26.2, R34.2, R42.2, R50.2, R58.2, R66.2, R74.2, U11.14 (OUT_D), U13.14 (OUT_D), U15.14 (OUT_D), U17.14 (OUT_D), U19.14 (OUT_D), U21.14 (OUT_D), U23.14 (OUT_D), U25.14 (OUT_D), U9.14 (OUT_D)
- net AY5: now also U6.5 (I4); no longer C16.2, C26.2, C36.2, C46.2, C59.2, C69.2, R14.2, R22.2, R30.2, R38.2, R46.2, U10.1 (OUT_A), U12.1 (OUT_A), U14.1 (OUT_A), U16.1 (OUT_A), U18.1 (OUT_A)
- net AY6: now also U6.4 (I5); no longer C11.2, C21.2, C31.2, C41.2, C54.2, C64.2, R11.2, R19.2, R27.2, R35.2, R43.2, U10.7 (OUT_B), U12.7 (OUT_B), U14.7 (OUT_B), U16.7 (OUT_B), U18.7 (OUT_B)
- net AY7: now also U6.3 (I6); no longer C18.2, C28.2, C38.2, C48.2, C61.2, R16.2, R24.2, R32.2, R40.2, R48.2, U10.8 (OUT_C), U12.8 (OUT_C), U14.8 (OUT_C), U16.8 (OUT_C), U18.8 (OUT_C)
- net AY8: now also U6.2 (I7); no longer C12.2, C22.2, C32.2, C42.2, C55.2, C65.2, R12.2, R20.2, R28.2, R36.2, R44.2, U10.14 (OUT_D), U12.14 (OUT_D), U14.14 (OUT_D), U16.14 (OUT_D), U18.14 (OUT_D)
- net GND: no longer C68.1
- net GNDREF: now also C64.1, C65.1, C68.1, C69.1, U20.12 (GND), U22.12 (GND), U5.12 (GND), U6.12 (GND)
- net Y1: no longer C14.1, C24.1, C34.1, C44.1, C57.1, C67.1, C77.1, C87.1, C97.1, R13.1, R21.1, R29.1, R37.1, R45.1, R53.1, R61.1, R69.1, R77.1, U11.2 (-IN_A), U13.2 (-IN_A), U15.2 (-IN_A), U17.2 (-IN_A), U19.2 (-IN_A), U21.2 (-IN_A), U23.2 (-IN_A), U25.2 (-IN_A), U9.2 (-IN_A)
- net Y2: no longer C19.1, C29.1, C39.1, C50.1, C62.1, C72.1, C82.1, C9.1, C92.1, R17.1, R25.1, R33.1, R41.1, R49.1, R57.1, R65.1, R73.1, R9.1, U11.6 (-IN_B), U13.6 (-IN_B), U15.6 (-IN_B), U17.6 (-IN_B), U19.6 (-IN_B), U21.6 (-IN_B), U23.6 (-IN_B), U25.6 (-IN_B), U9.6 (-IN_B)
- net Y3: no longer C100.1, C17.1, C27.1, C37.1, C47.1, C60.1, C70.1, C80.1, C90.1, R15.1, R23.1, R31.1, R39.1, R47.1, R55.1, R63.1, R71.1, R79.1, U11.9 (-IN_C), U13.9 (-IN_C), U15.9 (-IN_C), U17.9 (-IN_C), U19.9 (-IN_C), U21.9 (-IN_C), U23.9 (-IN_C), U25.9 (-IN_C), U9.9 (-IN_C)
- net Y4: no longer C10.1, C20.1, C30.1, C40.1, C52.1, C63.1, C73.1, C83.1, C93.1, R10.1, R18.1, R26.1, R34.1, R42.1, R50.1, R58.1, R66.1, R74.1, U11.13 (-IN_D), U13.13 (-IN_D), U15.13 (-IN_D), U17.13 (-IN_D), U19.13 (-IN_D), U21.13 (-IN_D), U23.13 (-IN_D), U25.13 (-IN_D), U9.13 (-IN_D)
- net Y5: no longer C16.1, C26.1, C36.1, C46.1, C59.1, C69.1, R14.1, R22.1, R30.1, R38.1, R46.1, U10.2 (-IN_A), U12.2 (-IN_A), U14.2 (-IN_A), U16.2 (-IN_A), U18.2 (-IN_A)
- net Y6: no longer C11.1, C21.1, C31.1, C41.1, C54.1, C64.1, R11.1, R19.1, R27.1, R35.1, R43.1, U10.6 (-IN_B), U12.6 (-IN_B), U14.6 (-IN_B), U16.6 (-IN_B), U18.6 (-IN_B)
- net Y7: no longer C18.1, C28.1, C38.1, C48.1, C61.1, R16.1, R24.1, R32.1, R40.1, R48.1, U10.9 (-IN_C), U12.9 (-IN_C), U14.9 (-IN_C), U16.9 (-IN_C), U18.9 (-IN_C)
- net Y8: no longer C12.1, C22.1, C32.1, C42.1, C55.1, C65.1, R12.1, R20.1, R28.1, R36.1, R44.1, U10.13 (-IN_D), U12.13 (-IN_D), U14.13 (-IN_D), U16.13 (-IN_D), U18.13 (-IN_D)
- new net AY10: C9.2, R9.2, U6.22 (I9), U9.7 (OUT_B)
- new net AY11: C17.2, R15.2, U6.21 (I10), U9.8 (OUT_C)
- new net AY12: C10.2, R10.2, U6.20 (I11), U9.14 (OUT_D)
- new net AY13: C16.2, R14.2, U10.1 (OUT_A), U6.19 (I12)
- new net AY14: C11.2, R11.2, U10.7 (OUT_B), U6.18 (I13)
- new net AY15: C18.2, R16.2, U10.8 (OUT_C), U6.17 (I14)
- new net AY16: C12.2, R12.2, U10.14 (OUT_D), U6.16 (I15)
- new net AY17: C24.2, R21.2, U11.1 (OUT_A), U20.9 (I0)
- new net AY18: C19.2, R17.2, U11.7 (OUT_B), U20.8 (I1)
- new net AY19: C27.2, R23.2, U11.8 (OUT_C), U20.7 (I2)
- new net AY20: C20.2, R18.2, U11.14 (OUT_D), U20.6 (I3)
- new net AY21: C26.2, R22.2, U12.1 (OUT_A), U20.5 (I4)
- new net AY22: C21.2, R19.2, U12.7 (OUT_B), U20.4 (I5)
- new net AY23: C28.2, R24.2, U12.8 (OUT_C), U20.3 (I6)
- new net AY24: C22.2, R20.2, U12.14 (OUT_D), U20.2 (I7)
- new net AY25: C34.2, R29.2, U13.1 (OUT_A), U20.23 (I8)
- new net AY26: C29.2, R25.2, U13.7 (OUT_B), U20.22 (I9)
- new net AY27: C37.2, R31.2, U13.8 (OUT_C), U20.21 (I10)
- new net AY28: C30.2, R26.2, U13.14 (OUT_D), U20.20 (I11)
- new net AY29: C36.2, R30.2, U14.1 (OUT_A), U20.19 (I12)
- new net AY30: C31.2, R27.2, U14.7 (OUT_B), U20.18 (I13)
- new net AY31: C38.2, R32.2, U14.8 (OUT_C), U20.17 (I14)
- new net AY32: C32.2, R28.2, U14.14 (OUT_D), U20.16 (I15)
- new net AY33: C44.2, R37.2, U15.1 (OUT_A), U22.9 (I0)
- new net AY34: C39.2, R33.2, U15.7 (OUT_B), U22.8 (I1)
- new net AY35: C47.2, R39.2, U15.8 (OUT_C), U22.7 (I2)
- new net AY36: C40.2, R34.2, U15.14 (OUT_D), U22.6 (I3)
- new net AY37: C46.2, R38.2, U16.1 (OUT_A), U22.5 (I4)
- new net AY38: C41.2, R35.2, U16.7 (OUT_B), U22.4 (I5)
- new net AY39: C48.2, R40.2, U16.8 (OUT_C), U22.3 (I6)
- new net AY40: C42.2, R36.2, U16.14 (OUT_D), U22.2 (I7)
- new net AY41: C57.2, R45.2, U17.1 (OUT_A), U22.23 (I8)
- new net AY42: C50.2, R41.2, U17.7 (OUT_B), U22.22 (I9)
- new net AY43: C60.2, R47.2, U17.8 (OUT_C), U22.21 (I10)
- new net AY44: C52.2, R42.2, U17.14 (OUT_D), U22.20 (I11)
- new net AY45: C59.2, R46.2, U18.1 (OUT_A), U22.19 (I12)
- new net AY46: C54.2, R43.2, U18.7 (OUT_B), U22.18 (I13)
- new net AY47: C61.2, R48.2, U18.8 (OUT_C), U22.17 (I14)
- new net AY48: C55.2, R44.2, U18.14 (OUT_D), U22.16 (I15)
- new net AY49: C67.2, R53.2, U19.1 (OUT_A), U5.9 (I0)
- new net AY50: C62.2, R49.2, U19.7 (OUT_B), U5.8 (I1)
- new net AY51: C70.2, R55.2, U19.8 (OUT_C), U5.7 (I2)
- new net AY52: C63.2, R50.2, U19.14 (OUT_D), U5.6 (I3)
- new net AY53: C77.2, R61.2, U21.1 (OUT_A), U5.5 (I4)
- new net AY54: C72.2, R57.2, U21.7 (OUT_B), U5.4 (I5)
- new net AY55: C80.2, R63.2, U21.8 (OUT_C), U5.3 (I6)
- new net AY56: C73.2, R58.2, U21.14 (OUT_D), U5.2 (I7)
- new net AY57: C87.2, R69.2, U23.1 (OUT_A), U5.23 (I8)
- new net AY58: C82.2, R65.2, U23.7 (OUT_B), U5.22 (I9)
- new net AY59: C90.2, R71.2, U23.8 (OUT_C), U5.21 (I10)
- new net AY60: C83.2, R66.2, U23.14 (OUT_D), U5.20 (I11)
- new net AY61: C97.2, R77.2, U25.1 (OUT_A), U5.19 (I12)
- new net AY62: C92.2, R73.2, U25.7 (OUT_B), U5.18 (I13)
- new net AY63: C100.2, R79.2, U25.8 (OUT_C), U5.17 (I14)
- new net AY64: C93.2, R74.2, U25.14 (OUT_D), U5.16 (I15)
- new net AY9: C14.2, R13.2, U6.23 (I8), U9.1 (OUT_A)
- new net EN-RIG-1-16: U6.15 (~{E})
- new net EN-RIG-17-32: U20.15 (~{E})
- new net EN-RIG-33-48: U22.15 (~{E})
- new net EN-RIG-49-64: U5.15 (~{E})
- new net RIG0: U20.10 (S0), U22.10 (S0), U5.10 (S0), U6.10 (S0)
- new net RIG1: U20.11 (S1), U22.11 (S1), U5.11 (S1), U6.11 (S1)
- new net RIG2: U20.14 (S2), U22.14 (S2), U5.14 (S2), U6.14 (S2)
- new net RIG3: U20.13 (S3), U22.13 (S3), U5.13 (S3), U6.13 (S3)
- new net Y10: C9.1, R9.1, U9.6 (-IN_B)
- new net Y11: C17.1, R15.1, U9.9 (-IN_C)
- new net Y12: C10.1, R10.1, U9.13 (-IN_D)
- new net Y13: C16.1, R14.1, U10.2 (-IN_A)
- new net Y14: C11.1, R11.1, U10.6 (-IN_B)
- new net Y15: C18.1, R16.1, U10.9 (-IN_C)
- new net Y16: C12.1, R12.1, U10.13 (-IN_D)
- new net Y17: C24.1, R21.1, U11.2 (-IN_A)
- new net Y18: C19.1, R17.1, U11.6 (-IN_B)
- new net Y19: C27.1, R23.1, U11.9 (-IN_C)
- new net Y20: C20.1, R18.1, U11.13 (-IN_D)
- new net Y21: C26.1, R22.1, U12.2 (-IN_A)
- new net Y22: C21.1, R19.1, U12.6 (-IN_B)
- new net Y23: C28.1, R24.1, U12.9 (-IN_C)
- new net Y24: C22.1, R20.1, U12.13 (-IN_D)
- new net Y25: C34.1, R29.1, U13.2 (-IN_A)
- new net Y26: C29.1, R25.1, U13.6 (-IN_B)
- new net Y27: C37.1, R31.1, U13.9 (-IN_C)
- new net Y28: C30.1, R26.1, U13.13 (-IN_D)
- new net Y29: C36.1, R30.1, U14.2 (-IN_A)
- new net Y30: C31.1, R27.1, U14.6 (-IN_B)
- new net Y31: C38.1, R32.1, U14.9 (-IN_C)
- new net Y32: C32.1, R28.1, U14.13 (-IN_D)
- new net Y33: C44.1, R37.1, U15.2 (-IN_A)
- new net Y34: C39.1, R33.1, U15.6 (-IN_B)
- new net Y35: C47.1, R39.1, U15.9 (-IN_C)
- new net Y36: C40.1, R34.1, U15.13 (-IN_D)
- new net Y37: C46.1, R38.1, U16.2 (-IN_A)
- new net Y38: C41.1, R35.1, U16.6 (-IN_B)
- new net Y39: C48.1, R40.1, U16.9 (-IN_C)
- new net Y40: C42.1, R36.1, U16.13 (-IN_D)
- new net Y41: C57.1, R45.1, U17.2 (-IN_A)
- new net Y42: C50.1, R41.1, U17.6 (-IN_B)
- new net Y43: C60.1, R47.1, U17.9 (-IN_C)
- new net Y44: C52.1, R42.1, U17.13 (-IN_D)
- new net Y45: C59.1, R46.1, U18.2 (-IN_A)
- new net Y46: C54.1, R43.1, U18.6 (-IN_B)
- new net Y47: C61.1, R48.1, U18.9 (-IN_C)
- new net Y48: C55.1, R44.1, U18.13 (-IN_D)
- new net Y49: C67.1, R53.1, U19.2 (-IN_A)
- new net Y50: C62.1, R49.1, U19.6 (-IN_B)
- new net Y51: C70.1, R55.1, U19.9 (-IN_C)
- new net Y52: C63.1, R50.1, U19.13 (-IN_D)
- new net Y53: C77.1, R61.1, U21.2 (-IN_A)
- new net Y54: C72.1, R57.1, U21.6 (-IN_B)
- new net Y55: C80.1, R63.1, U21.9 (-IN_C)
- new net Y56: C73.1, R58.1, U21.13 (-IN_D)
- new net Y57: C87.1, R69.1, U23.2 (-IN_A)
- new net Y58: C82.1, R65.1, U23.6 (-IN_B)
- new net Y59: C90.1, R71.1, U23.9 (-IN_C)
- new net Y60: C83.1, R66.1, U23.13 (-IN_D)
- new net Y61: C97.1, R77.1, U25.2 (-IN_A)
- new net Y62: C92.1, R73.1, U25.6 (-IN_B)
- new net Y63: C100.1, R79.1, U25.9 (-IN_C)
- new net Y64: C93.1, R74.1, U25.13 (-IN_D)
- new net Y9: C14.1, R13.1, U9.2 (-IN_A)
Other:
- moved on the sheet: C100, C62, C63, C66, C67, C70, C72, C73, C76, C77, C80, C82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
