File: Hardware/Schematics/04-Pilotaggio Matrice/04-Pilotaggio Matrice.kicad_sch (KiCad schematic)
At the start: 241 parts, among them J1 Conn_02x32_Odd_Even, J2 Conn_02x32_Odd_Even, J3 Conn_02x32_Odd_Even, U1 CD74HC4067M, U10 AD8604ARUZ, U11 AD8604ARUZ, U12 AD8604ARUZ, U13 AD8604ARUZ, U14 AD8604ARUZ, U15 AD8604ARUZ, U16 AD8604ARUZ, U17 AD8604ARUZ, U18 AD8604ARUZ, U19 AD8604ARUZ, U2 CD74HC4067M, U20 CD74HC4067M, U21 AD8604ARUZ, U22 CD74HC4067M, U23 AD8604ARUZ, U25 AD8604ARUZ, U3 CD74HC4067M, U4 CD74HC4067M, U5 CD74HC4067M, U6 CD74HC4067M, U69A AD8604ARUZ, U7 AD8604ARUZ, U8 AD8604ARUZ, U9 AD8604ARUZ

Commit message: update
Parts:
- added C71, C74, C75, C78: 56pF, symbol Device:C
- added R113, R114, R147, R148, R149, R150, R151, R152: 100K, symbol Device:R_US
- added R115, R117, R183, R184: 10k, symbol Device:R_US
- added R116, R118, R119, R120, R121, R122, R123, R124, R125, R126, R127, R128, R129, R130, R131, R132, R133, R134, R135, R136, R137, R138, R139, R140, R141, R142, R143, R144, R145, R146, R153, R154, R155, R156, R157, R158, R159, R160, R161, R162, R163, R164, R165, R166, R167, R168, R169, R170, R171, R172, R173, R174, R175, R176, R177, R178, R179, R180, R181, R182, R185, R186, R187, R188: 560, symbol Device:R_US
- added U24: LM339, symbol Comparator:LM339
- added U60D, U61D, U62D, U63D: AD8604ARUZ, AD8604ARUZ:SOP65P640X120-14N, symbol AD8604ARUZ:AD8604ARUZ
Connections:
- net +5V: now also R113.1, R147.1, R149.1, R151.1, U24.3 (V+)
- net AY1: now also R132.1
- net AY10: now also R141.1
- net AY11: now also R142.1
- net AY12: now also R143.1
- net AY13: now also R144.1
- net AY14: now also R145.1
- net AY15: now also R146.1
- net AY16: now also R186.1
- net AY17: now also R153.1
- net AY18: now also R154.1
- net AY19: now also R155.1
- net AY2: now also R133.1
- net AY20: now also R156.1
- net AY21: now also R157.1
- net AY22: now also R158.1
- net AY23: now also R159.1
- net AY24: now also R160.1
- net AY25: now also R161.1
- net AY26: now also R162.1
- net AY27: now also R163.1
- net AY28: now also R164.1
- net AY29: now also R165.1
- net AY3: now also R134.1
- net AY30: now also R166.1
- net AY31: now also R167.1
- net AY32: now also R188.1
- net AY33: now also R168.1
- net AY34: now also R169.1
- net AY35: now also R170.1
- net AY36: now also R171.1
- net AY37: now also R172.1
- net AY38: now also R173.1
- net AY39: now also R174.1
- net AY4: now also R135.1
- net AY40: now also R175.1
- net AY41: now also R176.1
- net AY42: now also R177.1
- net AY43: now also R178.1
- net AY44: now also R179.1
- net AY45: now also R180.1
- net AY46: now also R181.1
- net AY47: now also R182.1
- net AY48: now also R187.1
- net AY49: now also R122.1
- net AY5: now also R136.1
- net AY50: now also R123.1
- net AY51: now also R124.1
- net AY52: now also R125.1
- net AY53: now also R126.1
- net AY54: now also R121.1
- net AY55: now also R120.1
- net AY56: now also R116.1
- net AY57: now also R118.1
- net AY58: now also R119.1
- net AY59: now also R127.1
- net AY6: now also R137.1
- net AY60: now also R128.1
- net AY61: now also R129.1
- net AY62: now also R130.1
- net AY63: now also R131.1
- net AY64: now also R185.1
- net AY7: now also R138.1
- net AY8: now also R139.1
- net AY9: now also R140.1
- net GND: now also U24.12 (V-)
- net GNDREF: now also R114.2, R148.2, R150.2, R152.2
- new net: C75.1, R153.2, R154.2, R155.2, R156.2, R157.2, R158.2, R159.2, R160.2, R161.2, R162.2, R163.2, R164.2, R165.2, R166.2, R167.2, R183.1, R188.2, U62D.13 (-IN_D)
- new net: R149.2, R150.1, U62D.12 (+IN_D)
- new net: C71.1, R115.1, R116.2, R118.2, R119.2, R120.2, R121.2, R122.2, R123.2, R124.2, R125.2, R126.2, R127.2, R128.2, R129.2, R130.2, R131.2, R185.2, U60D.13 (-IN_D)
- new net: C78.1, R168.2, R169.2, R170.2, R171.2, R172.2, R173.2, R174.2, R175.2, R176.2, R177.2, R178.2, R179.2, R180.2, R181.2, R182.2, R184.1, R187.2, U63D.13 (-IN_D)
- new net: C74.1, R117.1, R132.2, R133.2, R134.2, R135.2, R136.2, R137.2, R138.2, R139.2, R140.2, R141.2, R142.2, R143.2, R144.2, R145.2, R146.2, R186.2, U61D.13 (-IN_D)
- new net: C71.2, R115.2, U24.7 (+), U60D.14 (OUT_D)
- new net: R113.2, R114.1, U60D.12 (+IN_D)
- new net: C78.2, R184.2, U24.9 (+), U63D.14 (OUT_D)
- new net: R147.2, R148.1, U61D.12 (+IN_D)
- new net: C74.2, R117.2, U24.5 (+), U61D.14 (OUT_D)
- new net: R151.2, R152.1, U63D.12 (+IN_D)
- new net: C75.2, R183.2, U24.11 (+), U62D.14 (OUT_D)

Commit message: update
Parts:
- added J5: Conn_02x25_Odd_Even, symbol Connector_Generic:Conn_02x25_Odd_Even
- added R189, R190, R191, R192, R193, R194, R195, R196, R197, R198, R199, R200, R201, R202, R204, R205: 100k, symbol Device:R_US
- added R203, R206, R207, R208: 2.2k, symbol Device:R_US
Connections:
- net +5V: now also R203.2, R206.2, R207.2, R208.2
- net COL0: now also J5.11 (Pin_11), R193.2
- net COL2: now also J5.15 (Pin_15), R195.2
- net COL3: now also J5.17 (Pin_17), R198.2
- net EN-COL-01-16: now also J5.1 (Pin_1), R189.2
- net EN-COL-17-32: now also J5.3 (Pin_3), R190.2
- net EN-COL-33-48: now also J5.5 (Pin_5), R191.2
- net EN-COL-49-64: now also J5.7 (Pin_7), R192.2
- net EN-RIG-17-32: now also J5.21 (Pin_21), R199.2
- net EN-RIG-33-48: now also J5.23 (Pin_23), R197.2
- net EN-RIG-49-64: now also J5.25 (Pin_25), R200.2
- net RIG0: now also J5.27 (Pin_27), R201.2
- net RIG1: now also J5.29 (Pin_29), R204.2
- net RIG2: now also J5.31 (Pin_31), R202.2
- net RIG3: now also J5.33 (Pin_33), R205.2
- net X10: now also J2.10 (Pin_10)
- net X11: now also J2.11 (Pin_11)
- net X12: now also J2.12 (Pin_12)
- net X13: now also J2.13 (Pin_13)
- net X14: now also J2.14 (Pin_14)
- net X15: now also J2.15 (Pin_15)
- net X16: now also J2.16 (Pin_16)
- net X17: now also J2.17 (Pin_17)
- net X18: now also J2.18 (Pin_18)
- net X19: now also J2.19 (Pin_19)
- net X2: now also J2.2 (Pin_2)
- net X20: now also J2.20 (Pin_20)
- net X21: now also J2.21 (Pin_21)
- net X22: now also J2.22 (Pin_22)
- net X23: now also J2.23 (Pin_23)
- net X24: now also J2.24 (Pin_24)
- net X25: now also J2.25 (Pin_25)
- net X26: now also J2.26 (Pin_26)
- net X27: now also J2.27 (Pin_27)
- net X29: now also J2.29 (Pin_29)
- net X30: now also J2.30 (Pin_30)
- net X31: now also J2.31 (Pin_31)
- net X32: now also J2.32 (Pin_32)
- net X33: now also J2.33 (Pin_33)
- net X34: now also J2.34 (Pin_34)
- net X35: now also J2.35 (Pin_35)
- net X36: now also J2.36 (Pin_36)
- net X37: now also J2.37 (Pin_37)
- net X38: now also J2.38 (Pin_38)
- net X39: now also J2.39 (Pin_39)
- net X4: now also J2.4 (Pin_4)
- net X40: now also J2.40 (Pin_40)
- net X41: now also J2.41 (Pin_41)
- net X42: now also J2.42 (Pin_42)
- net X43: now also J2.43 (Pin_43)
- net X44: now also J2.44 (Pin_44)
- net X45: now also J2.45 (Pin_45)
- net X46: now also J2.46 (Pin_46)
- net X47: now also J2.47 (Pin_47)
- net X48: now also J2.48 (Pin_48)
- net X49: now also J2.49 (Pin_49)
- net X50: now also J2.50 (Pin_50)
- net X51: now also J2.51 (Pin_51)
- net X52: now also J2.52 (Pin_52)
- net X53: now also J2.53 (Pin_53)
- net X54: now also J2.54 (Pin_54)
- net X55: now also J2.55 (Pin_55)
- net X56: now also J2.56 (Pin_56)
- net X57: now also J2.57 (Pin_57)
- net X58: now also J2.58 (Pin_58)
- net X59: now also J2.59 (Pin_59)
- net X6: now also J2.6 (Pin_6)
- net X60: now also J2.60 (Pin_60)
- net X61: now also J2.61 (Pin_61)
- net X62: now also J2.62 (Pin_62)
- net X63: now also J2.63 (Pin_63)
- net X64: now also J2.64 (Pin_64)
- net X7: now also J2.7 (Pin_7)
- net X8: now also J2.8 (Pin_8)
- net X9: now also J2.9 (Pin_9)
- net Y10: no longer J2.10 (Pin_10)
- net Y11: no longer J2.11 (Pin_11)
- net Y12: no longer J2.12 (Pin_12)
- net Y13: no longer J2.13 (Pin_13)
- net Y14: no longer J2.14 (Pin_14)
- net Y15: no longer J2.15 (Pin_15)
- net Y16: no longer J2.16 (Pin_16)
- net Y17: no longer J2.17 (Pin_17)
- net Y18: no longer J2.18 (Pin_18)
- net Y19: no longer J2.19 (Pin_19)
- net Y2: no longer J2.2 (Pin_2)
- net Y20: no longer J2.20 (Pin_20)
- net Y21: no longer J2.21 (Pin_21)
- net Y22: no longer J2.22 (Pin_22)
- net Y23: no longer J2.23 (Pin_23)
- net Y24: no longer J2.24 (Pin_24)
- net Y25: no longer J2.25 (Pin_25)
- net Y26: no longer J2.26 (Pin_26)
- net Y27: no longer J2.27 (Pin_27)
- net Y29: no longer J2.29 (Pin_29)
- net Y30: no longer J2.30 (Pin_30)
- net Y31: no longer J2.31 (Pin_31)
- net Y32: no longer J2.32 (Pin_32)
- net Y33: no longer J2.33 (Pin_33)
- net Y34: no longer J2.34 (Pin_34)
- net Y35: no longer J2.35 (Pin_35)
- net Y36: no longer J2.36 (Pin_36)
- net Y37: no longer J2.37 (Pin_37)
- net Y38: no longer J2.38 (Pin_38)
- net Y39: no longer J2.39 (Pin_39)
- net Y4: no longer J2.4 (Pin_4)
- net Y40: no longer J2.40 (Pin_40)
- net Y41: no longer J2.41 (Pin_41)
- net Y42: no longer J2.42 (Pin_42)
- net Y43: no longer J2.43 (Pin_43)
- net Y44: no longer J2.44 (Pin_44)
- net Y45: no longer J2.45 (Pin_45)
- net Y46: no longer J2.46 (Pin_46)
- net Y47: no longer J2.47 (Pin_47)
- net Y48: no longer J2.48 (Pin_48)
- net Y49: no longer J2.49 (Pin_49)
- net Y50: no longer J2.50 (Pin_50)
- net Y51: no longer J2.51 (Pin_51)
- net Y52: no longer J2.52 (Pin_52)
- net Y53: no longer J2.53 (Pin_53)
- net Y54: no longer J2.54 (Pin_54)
- net Y55: no longer J2.55 (Pin_55)
- net Y56: no longer J2.56 (Pin_56)
- net Y57: no longer J2.57 (Pin_57)
- net Y58: no longer J2.58 (Pin_58)
- net Y59: no longer J2.59 (Pin_59)
- net Y6: no longer J2.6 (Pin_6)
- net Y60: no longer J2.60 (Pin_60)
- net Y61: no longer J2.61 (Pin_61)
- net Y62: no longer J2.62 (Pin_62)
- net Y63: no longer J2.63 (Pin_63)
- net Y64: no longer J2.64 (Pin_64)
- net Y7: no longer J2.7 (Pin_7)
- net Y8: no longer J2.8 (Pin_8)
- net Y9: no longer J2.9 (Pin_9)
- net actv-1-16: now reaches U24.2
- net actv-1-16: now also J5.22 (Pin_22), R203.1
- net Tp-Vthr: now reaches U24.4 (-)
- net Tp-Vthr: now also U24.10 (-), U24.6 (-), U24.8 (-), J5.32 (Pin_32)
- net actv-17-32: now reaches U24.13
- net actv-17-32: now also J5.24 (Pin_24), R206.1
- net actv-33-48: now reaches U24.14
- net actv-33-48: now also J5.26 (Pin_26), R207.1
- net actv-49-64: now reaches U24.1
- net actv-49-64: now also J5.28 (Pin_28), R208.1
- new net: R189.1, R190.1, R191.1, R192.1, R193.1, R194.1, R195.1, R196.1, R197.1, R198.1, R199.1, R200.1, R201.1, R202.1, R204.1, R205.1
- new net ADC1: J5.4 (Pin_4)
- new net ADC2: J5.6 (Pin_6)
- new net ADC3: J5.8 (Pin_8)
- new net ADC4: J5.10 (Pin_10)
- new net COl1: J5.13 (Pin_13), R194.2
- new net EN-COL-113-128: J5.18 (Pin_18)
- new net EN-COL-65-80: J5.12 (Pin_12)
- new net EN-COL-81-96: J5.14 (Pin_14)
- new net EN-COL-97-112: J5.16 (Pin_16)
- new net EN-RIG-01-16: J5.19 (Pin_19), R196.2
Other:
- moved on the sheet: U24A, U24B, U24C, U24D

Commit message: finalized the schematic conversion
Parts:
- added C79, C81, C84, C85: 470pF, symbol Device:C
- added J4: Conn_02x12_Odd_Even, symbol Connector_Generic:Conn_02x12_Odd_Even
- added R209, R214, R215, R216: 330, symbol Device:R_US
- added R210, R211, R212, R213: 560, symbol Device:R_US
- added TP1, TP2: ADC4, symbol Connector:TestPoint
- added TP3: ADC1, symbol Connector:TestPoint
- added TP4: ADC2, symbol Connector:TestPoint
Connections:
- net ADC2 is gone; now on net ADC1: J5.6 (Pin_6)
- net ADC3 is gone; now on net ADC1: J5.8 (Pin_8)
- net +5V: now also J5.35 (Pin_35), J5.37 (Pin_37), J5.39 (Pin_39), J4.17 (Pin_17), J4.19 (Pin_19)
- net ADC1: now also C79.2, C81.2, C84.2, R209.2, R214.2, R215.2, TP1.1, TP4.1
- net COL0: now also J4.1 (Pin_1)
- net COL2: now also J4.5 (Pin_5)
- net COL3: now also J4.7 (Pin_7)
- net COl1: now also J4.3 (Pin_3)
- net EN-COL-113-128: now also J4.15 (Pin_15), R213.1
- net EN-COL-65-80: now also J4.9 (Pin_9), R210.1
- net EN-COL-81-96: now also J4.11 (Pin_11), R211.1
- net EN-COL-97-112: now also J4.13 (Pin_13), R212.1
- net GND: now also J5.45 (Pin_45), J5.47 (Pin_47), J5.49 (Pin_49), C79.1, C81.1, C84.1, C85.1, J4.22 (Pin_22), J4.24 (Pin_24)
- net GNDREF: now also J5.46 (Pin_46), J5.48 (Pin_48), J5.50 (Pin_50), J4.21 (Pin_21), J4.23 (Pin_23), R210.2, R211.2, R212.2, R213.2
- net at U22.1 (COM): now also R209.1
- net at U6.1 (COM): now also R215.1
- net +8V: now reaches J5.40 (Pin_40)
- net +8V: now also J5.42 (Pin_42), J5.44 (Pin_44)
- net at U5.1 (COM): now also R216.1
- net at U20.1 (COM): now also R214.1
- net ADC4: no longer names the net of J5.10 (Pin_10)
- net ADC4: now also C85.2, R216.2, TP2.1, TP3.1
