File: Hardware/Schematics/01-Micro STM32/01-Micro STM32.kicad_sch (KiCad schematic)
At the start: 0 parts

Commit message: update
Parts:
- added J1: Screw_Terminal_01x04, symbol Connector:Screw_Terminal_01x04
- added U1: MCP23017_ML, Package_DFN_QFN:QFN-28-1EP_6x6mm_P0.65mm_EP4.25x4.25mm, symbol Interface_Expansion:MCP23017_ML
- added U2: ESP32-DEVKITC-32D, ESP32-DEVKITC-32D:MODULE_ESP32-DEVKITC-32D, symbol ESP32-DEVKITC-32D:ESP32-DEVKITC-32D
- added U3, U4: 74HCT138, symbol 74xx:74HCT138
- added U69A: AD8604ARUZ, AD8604ARUZ:SOP65P640X120-14N, symbol AD8604ARUZ:AD8604ARUZ

Commit message: update
Parts:
- added C1: 47pF, symbol Device:C_Small
- added C2: 100nF, symbol Device:C_Small
- added J2: Conn_01x12_MountingPin, symbol Connector_Generic_MountingPin:Conn_01x12_MountingPin
- added R1: 27Ω, symbol Device:R_US
- added R2: 22Ω, symbol Device:R_US
- added SW1: SW_DIP_x05, symbol Switch:SW_DIP_x05
- added U5: CP2102N-Axx-xQFN28, Package_DFN_QFN:QFN-28-1EP_5x5mm_P0.5mm_EP3.35x3.35mm, symbol Interface_USB:CP2102N-Axx-xQFN28
- added U6: USBLC6-2SC6, Package_TO_SOT_SMD:SOT-23-6, symbol Power_Protection:USBLC6-2SC6
Connections:
- net RXD: now reaches U2.J2-16 (SD2)
- net RXD: now also U5.25 (RXD)
- net TXD: now reaches U2.J2-17 (SD3)
- net TXD: now also U5.26 (TXD)
- net CTS: now reaches U2.J2-18 (CMD)
- net CTS: now also U5.23 (~{CTS})
- net +5V: now reaches U2.J2-19 (EXT_5V)
- net +5V: now also U1.9 (VDD), J2.1 (Pin_1), J2.2 (Pin_2)
- net GNDREF: now reaches U2.J3-1 (GND3)
- net GNDREF: now also U1.10 (VSS), U2.J3-7 (GND2), J2.11 (Pin_11), J2.12 (Pin_12)
- net at U2.J3-10 (IO5): now also J2.4 (Pin_4)
- net at U2.J3-11 (IO17): now also J2.3 (Pin_3)
- net ADC1: now reaches U2.J3-12 (IO16)
- net ADC2: now reaches U2.J3-13 (IO4)
- net ADC3: now reaches U2.J3-14 (IO0)
- net CS-SD: now reaches U2.J3-15 (IO2)
- net I2C_SCL: now reaches U2.J3-17 (SD1)
- net I2C_SCL: now also U1.13 (SDA)
- net I2C_SDA: now reaches U2.J3-18 (SD0)
- net I2C_SDA: now also U1.12 (SCK)
- net RTS: now reaches U2.J3-19 (CLK)
- net RTS: now also U5.24 (~{RTS})
- net at U2.J3-2 (IO23): now also J2.7 (Pin_7)
- net at U2.J3-8 (IO19): now also J2.6 (Pin_6)
- net at U2.J3-9 (IO18): now also J2.5 (Pin_5)
- net GPB0: now reaches U1.1 (GPB0)
- net GPB1: now reaches U1.2 (GPB1)
- net at U1.24 (GPA3): now also SW1.6
- net at U1.25 (GPA4): now also SW1.7
- net at U1.26 (GPA5): now also SW1.8
- net at U1.27 (GPA6): now also SW1.9
- net at U1.28 (GPA7): now also SW1.10
- net GPB3: now reaches U1.4 (GPB3)
- new net: R2.1, U6.4 (I/O2)
- new net: R2.2, U5.4 (D+)
- new net: R1.1, U6.6 (I/O1)
- new net: C1.2, R1.2, U5.5 (D-)
- new net +5V_USB: C2.2, U5.7 (VREGIN), U5.8 (VBUS), U6.5 (VBUS)
- new net GND: C1.1, C2.1, SW1.1, SW1.2, SW1.3, SW1.4, SW1.5, U5.29 (GND), U5.3 (GND), U6.2 (GND)
Other:
- moved on the sheet: U1, U2, U4, U69A

Commit message: update
Parts:
- added C3: 100nF, symbol Device:C_Small
- added J3: Conn_02x25_Odd_Even, symbol Connector_Generic:Conn_02x25_Odd_Even
- added JP1, JP2: Jumper_2_Open, symbol Jumper:Jumper_2_Open
- added R3, R4, R5: 100KΩ, symbol Device:R_US
- added R6: 4K7Ω, symbol Device:R_US
- added R7: 100kΩ, symbol Device:R_US
- added TP1: TestPoint, symbol Connector:TestPoint
Connections:
- net +5V: now also JP1.1 (A)
- net GND: now also U69A.11 (V-), C3.2, R5.1, R7.1
- net GNDREF: now also U2.J2-14 (GND1)
- net ADC4: now reaches U2.J2-11 (IO27)
- net MTMS/SCK: now reaches U2.J2-12 (IO14)
- net MTDI/MISO: now reaches U2.J2-13 (IO12)
- net MTCK/MOSI: now reaches U2.J2-15 (IO13)
- net actv-49-64: now reaches U2.J2-3 (SENSOR_VP)
- net actv-49-64: now also J3.28 (Pin_28)
- net actv-33-48: now reaches U2.J2-4 (SENSOR_VN)
- net actv-33-48: now also J3.26 (Pin_26)
- net actv-17-32: now reaches U2.J2-5 (IO34)
- net actv-17-32: now also J3.24 (Pin_24)
- net actv-1-16: now reaches U2.J2-6 (IO35)
- net actv-1-16: now also J3.22 (Pin_22)
- net DAC1: now reaches U2.J2-9 (IO25)
- net DAC1: now also R3.1
- net at U69A.12 (+IN_D): now also R3.2
- net at U69A.13 (-IN_D): now also R4.2, R5.2
- net at U69A.14 (OUT_D): now also JP2.1 (A), R4.1
- net +8V: now reaches U69A.4 (V+)
- net +8V: now also C3.1
- new net: JP1.2 (B), JP2.2 (B), R6.1
- new net: J3.32 (Pin_32), R6.2, R7.2, TP1.1
Other:
- moved on the sheet: U3, U69A

Commit message: update
Connections:
- net +8V: now also J3.40 (Pin_40), J3.42 (Pin_42), J3.44 (Pin_44)
- net ADC1: now also J3.4 (Pin_4)
- net ADC2: now also J3.6 (Pin_6)
- net ADC3: now also J3.8 (Pin_8)
- net ADC4: now also J3.10 (Pin_10)
- net GND: now also J3.45 (Pin_45), J3.47 (Pin_47), J3.49 (Pin_49)
- net GNDREF: now also J3.46 (Pin_46), J3.48 (Pin_48), J3.50 (Pin_50)
- net EN-RIG-65-80: now reaches U4.12 (~{Y3})
- net EN-RIG-65-80: now also J3.25 (Pin_25)
- net EN-RIG-49-64: now reaches U4.13 (~{Y2})
- net EN-RIG-49-64: now also J3.23 (Pin_23)
- net EN-RIG-33-48: now reaches U4.14 (~{Y1})
- net EN-RIG-33-48: now also J3.21 (Pin_21)
- net EN-RIG-01-16: now reaches U4.15 (~{Y0})
- net EN-RIG-01-16: now also J3.19 (Pin_19)
- net EN-COL-01-16: now reaches J3.1 (Pin_1)
- net EN-COL-01-16: now also U3.15 (~{Y0})
- net COL0: now reaches J3.11 (Pin_11)
- net EN-COL-65-80: now reaches J3.12 (Pin_12)
- net EN-COL-65-80: now also U3.11 (~{Y4})
- net COL1: now reaches J3.13 (Pin_13)
- net EN-COL-81-96: now reaches J3.14 (Pin_14)
- net EN-COL-81-96: now also U3.10 (~{Y5})
- net COL2: now reaches J3.15 (Pin_15)
- net EN-COL-97-112: now reaches J3.16 (Pin_16)
- net EN-COL-97-112: now also U3.9 (~{Y6})
- net COL3: now reaches J3.17 (Pin_17)
- net EN-COL-113-128: now reaches J3.18 (Pin_18)
- net EN-COL-113-128: now also U3.7 (~{Y7})
- net GPB5: now reaches J3.2 (Pin_2)
- net RIG0: now reaches J3.27 (Pin_27)
- net RIG1: now reaches J3.29 (Pin_29)
- net EN-COL-17-32: now reaches J3.3 (Pin_3)
- net EN-COL-17-32: now also U3.14 (~{Y1})
- net RIG2: now reaches J3.31 (Pin_31)
- net RIG3: now reaches J3.33 (Pin_33)
- net +3V3: now reaches J3.35 (Pin_35)
- net +3V3: now also J3.37 (Pin_37), J3.39 (Pin_39)
- net GPB9: now reaches J3.41 (Pin_41)
- net EN-COL-33-48: now reaches J3.5 (Pin_5)
- net EN-COL-33-48: now also U3.13 (~{Y2})
- net EN-COL-49-64: now reaches J3.7 (Pin_7)
- net EN-COL-49-64: now also U3.12 (~{Y3})
Other:
- moved on the sheet: C1, C2, C3, J1, J2, J3, JP1, JP2, R1, R2, R3, R4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

Commit message: update
Parts:
- removed J1: Screw_Terminal_01x04, symbol Connector:Screw_Terminal_01x04
- removed J2: Conn_01x12_MountingPin, symbol Connector_Generic_MountingPin:Conn_01x12_MountingPin
- added C4: 47uF, symbol Device:C_Polarized_Small_US
- added D1: LED_0, symbol Device:LED
- added D2: D_Zener, symbol Device:D_Zener
- added J1: Conn_01x06, symbol Connector_Generic:Conn_01x06
- added J4: Conn_01x04, symbol Connector_Generic:Conn_01x04
- added J5: Conn_01x12, symbol Connector_Generic:Conn_01x12
- added J6: Micro_SD_Card_Det1, symbol Connector:Micro_SD_Card_Det1
- added L1: 470nH, symbol Device:L
- added Q1: BC817, Package_TO_SOT_SMD:SOT-23, symbol Transistor_BJT:BC817
- added R10, R12: 1KΩ, symbol Device:R_US
- added R11: 100Ω, symbol Device:R_US
- added R13, R14, R9: 10KΩ, symbol Device:R_US
- added R8: 1kΩ, symbol Device:R_US
- added U7: 74HC04, symbol 74xx:74HC04
Connections:
- net +3V3: now also D1.2 (A), J4.4 (Pin_4), L1.1, R13.1, R14.1
- net +5V: now also J5.1 (Pin_1), R12.1, R9.2
- net GND: now also C4.1, D2.2 (A), J1.1 (Pin_1), J4.1 (Pin_1), Q1.2 (E), U7.11, U7.13
- net GNDREF: now also U3.4 (~{E0}), U3.5 (~{E1}), U3.6 (E2), U4.4 (~{E0}), U4.5 (~{E1}), U4.6 (E2), J5.10 (Pin_10), J5.11 (Pin_11), J5.12 (Pin_12)
- net GPB0: now also R8.1
- net GPB5: now also U7.1, U7.4
- net I2C_SCL: now also J4.3 (Pin_3)
- net I2C_SDA: now also J4.2 (Pin_2)
- net MTCK/MOSI: now also J6.3 (CMD)
- net MTDI/MISO: now also J6.7 (DAT0), R14.2
- net MTMS/SCK: now also J6.5 (CLK)
- net at U2.J3-10 (IO5): now also J5.3 (Pin_3)
- net at U2.J3-11 (IO17): now also J5.2 (Pin_2)
- net at U2.J3-2 (IO23): now also J5.6 (Pin_6)
- net at U2.J3-8 (IO19): now also J5.5 (Pin_5)
- net at U2.J3-9 (IO18): now also J5.4 (Pin_4)
- new net: J1.3 (Pin_3), R12.2, U7.9
- new net: J1.5 (Pin_5), R10.1, U7.2
- new net: Q1.1 (B), R10.2
- new net: D1.1 (K), R8.2
- new net: D2.1 (K), R11.1, U7.3
- new net: J1.4 (Pin_4), R11.2
- new net: C4.2, J6.4 (VDD), L1.2
- new net: J6.8 (DAT1), R13.2
- new net: J1.6 (Pin_6), Q1.3 (C), R9.1

Commit message: update
Parts:
- added C5: 10uF, symbol Device:C_Polarized_Small_US
- added C6: 100nF, symbol Device:C_Small
- added D3: LED, symbol Device:LED
- added J10: USB_B_Mini, symbol Connector:USB_B_Mini
- added J2: Conn_02x05_Odd_Even, symbol Connector_Generic:Conn_02x05_Odd_Even
- added J9: USB_B, symbol Connector:USB_B
- added JP3: Jumper_2_Open, symbol Jumper:Jumper_2_Open
- added R15, R16: 10KΩ, symbol Device:R_US
- added U8: LM1117MP-3.3, Package_TO_SOT_SMD:SOT-223-3_TabPin2, symbol Regulator_Linear:LM1117MP-3.3
Connections:
- net +3V3: now also R15.1
- net +5V_USB: now also J10.1 (VBUS), J9.1 (VBUS), JP3.1 (A)
- net CS-SD: now also J6.2 (DAT3/CD)
- net GND: now also J10.5 (GND), J2.3 (Pin_3), J2.5 (Pin_5), J2.7 (Pin_7), J2.9 (Pin_9), J9.4 (GND)
- net MTCK/MOSI: now also J2.4 (Pin_4)
- net MTDI/MISO: now also J2.8 (Pin_8)
- net MTMS/SCK: now also J2.2 (Pin_2)
- net at U6.1 (I/O1): now also J10.2 (D-), J9.2 (D-)
- net at U6.3 (I/O2): now also J10.3 (D+), J9.3 (D+)
- net at J6.1 (DAT2): now also R15.2
- new net: J2.1 (Pin_1), JP3.2 (B)
- new net TDO: J2.6 (Pin_6)
- no-connect marks 0 -> 1

Commit message: update
Parts:
- added U10: BQ25172DSGR, BQ25172DSGR:IC_BQ25172DSGR, symbol BQ25172DSGR:BQ25172DSGR
- added U11: LDL112-LD0, BQ25172DSGR:IC_BQ25172DSGR, symbol LDL112D18R:LDL112-LD0
- R16: value 10KΩ -> 560Ω
Connections:
- net +3V3: now also C5.1, C6.1, D3.2 (A), U8.2 (VO)
- net GND: now also C5.2, C6.2, R16.1, U8.1 (GND), U11.2 (GND), U11.3 (GND), U11.6 (GND), U11.7 (GND)
- net at U8.3 (VI): now also U11.4 (Vin)
- net at D3.1 (K): now also R16.2
Other:
- moved on the sheet: C5, C6, D3, R16

Commit message: Finalized Schematic
Parts:
- added C10: 100uF, symbol Device:C_Polarized_Small_US
- added C11: 4.7nF, symbol Device:C_Small
- added C7, C8: 10uF, symbol Device:C_Polarized_Small_US
- added C9: 100nF, symbol Device:C_Small
- added D4: LED, symbol Device:LED
- added D5: GBU8A, Diode_THT:Diode_Bridge_Vishay_GBU, symbol Diode_Bridge:GBU8A
- added D6: D_Schottky, symbol Device:D_Schottky
- added IC1, IC2: 74HCT4040, 74HCT4040:TSSOP16, symbol 74HCT4040:74HCT4040
- added J11: Jack-DC, symbol Connector:Jack-DC
- added J12: RF-Sync-Tx, symbol Connector_Generic:Conn_01x04
- added J13: RF-Sync-Rx, symbol Connector_Generic:Conn_01x04
- added J7, J8: Conn_01x02, symbol Connector_Generic:Conn_01x02
- added Q2: BC817, Package_TO_SOT_SMD:SOT-23, symbol Transistor_BJT:BC817
- added Q3: IRF9540N, Package_TO_SOT_THT:TO-220-3_Vertical, symbol Transistor_FET:IRF9540N
- added R17, R18: 560Ω, symbol Device:R_US
- added R19: 100Ω, symbol Device:R_US
- added R20, R21, R22, R23, R25: 10kΩ, symbol Device:R_US
- added R24: 1kΩ, symbol Device:R_US
- added R26: 2.2kΩ, symbol Device:R_US
- added SW2: SW_Push, symbol Switch:SW_Push
- added TH1: Thermistor_PTC, symbol Device:Thermistor_PTC
- added TP2: TP-V5V, symbol Connector:TestPoint
- added TP3: TP-GND, symbol Connector:TestPoint
Connections:
- net +3V3: now also Q3.3 (S), R26.2
- net +5V: now also U11.1 (Vout), C8.1, C9.1, IC1.16 (VCC), IC2.16 (VCC), R17.2, TP2.1
- net +5V_USB: now also D6.2 (A), R19.1, R21.1
- net +8V: now also U10.8 (OUT), J7.2 (Pin_2), J8.2 (Pin_2), SW2.1
- net COL0: now also IC1.9 (Q0)
- net COL1: now also IC1.7 (Q1)
- net COL2: now also U3.16 (VCC), IC1.6 (Q2)
- net COL3: now also IC1.5 (Q3)
- net GND: now also U10.4 (GND), C10.2, C11.2, C7.2, C8.2, C9.2, D5.4 (-), IC1.8 (GND), IC2.8 (GND), J12.2 (Pin_2), J13.4 (Pin_4), J7.1 (Pin_1), Q2.2 (E), R18.1, R22.1, R23.1, R24.2, R25.2, TP3.1
- net GNDREF: now also U4.3 (A2), IC2.4 (Q6)
- net GPB1: now also J12.3 (Pin_3)
- net GPB3: now also Q3.1 (G), R26.1
- net RIG0: now also IC2.9 (Q0)
- net RIG1: now also IC2.7 (Q1)
- net RIG2: now also IC2.6 (Q2)
- net RIG3: now also IC2.5 (Q3)
- net at U11.4 (Vin), U8.3 (VI): now also C7.1, J8.1 (Pin_1), SW2.2
- net GPB6: now reaches U11.5 (en)
- net at U11.8 (ADJ): now also R17.1, R18.2
- net at U4.1 (A0): now also IC2.3 (Q4)
- net at U4.2 (A1): now also IC2.2 (Q5)
- net at JP2.1 (A), R4.1, U69A.14 (OUT_D): now also J3.32 (Pin_32), R6.2, R7.2, TP1.1
- net at U7.5: now also U10.5 (STAT), R21.2
- net at U7.6: now also R20.2
- net at U10.1 (IN): now also C10.1, C11.1, D5.1 (+), D6.1 (K)
- net at U10.2 (ISET): now also R24.1
- net at U10.3 (TS): now also R25.1
- net at U10.6 (TMR): now also R23.2
- net at U10.7 (VSET): now also R22.2
- net at U3.1 (A0): now also IC1.3 (Q4)
- net at U3.2 (A1): now also IC1.2 (Q5)
- net at U3.3 (A2): now also IC1.4 (Q6)
- new net: J12.1 (Pin_1), J13.1 (Pin_1), Q3.2 (D)
- new net: D4.1 (K), Q2.3 (C)
- new net: D4.2 (A), R19.2
- new net: Q2.1 (B), R20.1
- new net: D5.2, TH1.2
- new net: D5.3, J11.2
- new net: J11.1, TH1.1
- new net GPB2: J13.2 (Pin_2)
Other:
- note added: "5 amp bridge"
- moved on the sheet: C5, C6, D3, R16, U10, U8
